File: Arduino_Workshop_Files/Workshop_Schematics/Workshop_000.sch (EAGLE design)
At the start: 22 parts

Commit message: Updated Arduino Sketches
Parts:
- added D1, D2, D3, D4: (no value), adafruit:DIODEDO-1N4148
- added OP-AMP: MCP6021T-E/OT, SparkFun-IC-Amplifiers:MCP6021T-E/OT
- added POT: (no value), adafruit:TRIMPOT3386
- added R11, R12, R14, R15, R16: 1k, rcl:R-US_R0805
- added R13: 10k, rcl:R-US_R0805
- added S5, S6, S7, S8: (no value), SparkFun-Switches:MOMENTARY-SWITCH-SPST-2-SMD-5.2MM
Connections:
- new net +3V3: POT.E
- new net A0: OP-AMPG1.OUT, R11.1, R13.1, R14.2
- new net N$10: D2.A, S8.4
- new net N$11: D4.A, S7.4
- new net N$12: D3.A, S6.3, S6.4
- new net N$13: S5.2, S6.2
- new net N$14: S7.2, S8.2
- new net N$7: OP-AMPG1.-IN, POT.A, R11.2, R12.2
- new net N$8: OP-AMPG1.+IN, POT.S
- new net N$9: D1.A, S5.4
- new net VIN: R13.2
- net GND: now also R12.1, R14.1, R15.2, R16.2
- net PIN2: now also S5.1
- net PIN3: now also S8.1
- net PIN4: now also D1.C, D2.C, R16.1
- net PIN5: now also D3.C, D4.C, R15.1
Other:
- note added: "BUTTON MATRIX"
- note added: "Non-Inverting Op-Amp"
- note added: "PULL-DOWN"
- note added: "PULL-UP"
- note added: "USE PIN 2, 3 FOR ROW USE PIN 4, 5 FOR COLUMN"
- note added: "Voltage Divider"
- note removed: "USE PIN 1, 2 FOR ROW USE PIN 3, 4 FOR COLUMN"
- moved on the sheet: LED1, LED2, LED3, LED4, R1, R2
